File: StepperBoard/StepperBoard.brd (EAGLE design)
At the start: 210.3 x 100.2 mm, 129 parts, among them J1 F-2X18-DIL-100, U1 A4988_STEPPER_MOTOR_DRIVER_CA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, U10 A4988_STEPPER_MOTOR_DRIVER_CA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, U11 A4988_STEPPER_MOTOR_DRIVER_CA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, U12 A4988_STEPPER_MOTOR_DRIVER_CA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, U13 A4988_STEPPER_MOTOR_DRIVER_CA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, U14 A4988_STEPPER_MOTOR_DRIVER_CA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, U15 A4988_STEPPER_MOTOR_DRIVER_CA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, U2 A4988_STEPPER_MOTOR_DRIVER_CA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, U3 A4988_STEPPER_MOTOR_DRIVER_CA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, U4 A4988_STEPPER_MOTOR_DRIVER_CA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, U5 A4988_STEPPER_MOTOR_DRIVER_CA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, U6 A4988_STEPPER_MOTOR_DRIVER_CA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, U7 A4988_STEPPER_MOTOR_DRIVER_CA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, U8 A4988_STEPPER_MOTOR_DRIVER_CA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, U9 A4988_STEPPER_MOTOR_DRIVER_CA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

Commit message: Add files via upload
Board design updated
Parts:
- removed J10, J11, J12, J13, J14, J15, J16, J2, J3, J4, J5, J6, J7, J8, J9: (no value), SparkFun-Connectors:1X02_2.54_SCREWTERM
- removed R1, R11, R13, R15, R17, R19, R26, R28, R3, R30, R37, R39, R5, R7, R9: 4.7k, SparkFun-Resistors:0603
- added JP10, JP11, JP12, JP13, JP14, JP15, JP17, JP18, JP19, JP20, JP5, JP6, JP7, JP8, JP9: (no value), pinhead:1X01
- moved X2 197.6 mm to (217.6, 12.3)
- moved R10 145.0 mm to (49.2, 51.4)
- moved R2 145.0 mm to (8.39, 51.2)
- moved R4 145.0 mm to (18.7, 51.4)
- moved R6 145.0 mm to (28.9, 51.4)
- moved R8 145.0 mm to (38.8, 51.4)
- moved SW1 145.0 mm to (8.44, 59.3)
- moved SW2 145.0 mm to (18.6, 59.3)
- moved SW3 145.0 mm to (28.8, 59.3)
- moved SW4 145.0 mm to (38.9, 59.3)
- moved SW5 145.0 mm to (49.1, 59.3)
- moved R12 144.9 mm to (8.26, 35.4)
- moved R14 144.9 mm to (18.7, 35.4)
- moved R16 144.9 mm to (28.6, 35.2)
- moved R18 144.9 mm to (38.8, 35.2)
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Connections:
- removed net N$101: J14.P1, R15.2, U5.5
- removed net N$103: J15.P1, R17.2, U4.5
- removed net N$105: J16.P1, R19.2, U6.5
- removed net N$124: J6.P1, R9.2, U3.5
- removed net N$151: J7.P1, R26.2, U14.5
- removed net N$153: J8.P1, R28.2, U15.5
- removed net N$155: J9.P1, R30.2, U12.5
- removed net N$157: J10.P1, R37.2, U11.5
- removed net N$159: J11.P1, R39.2, U13.5
- removed net N$35: J3.P1, R3.2, U8.5
- removed net N$37: J4.P1, R5.2, U2.5
- removed net N$8: J2.P1, R1.2, U7.5
- removed net N$81: J5.P1, R7.2, U1.5
- removed net N$97: J12.P1, R11.2, U9.5
- removed net N$99: J13.P1, R13.2, U10.5
- net N$1: no longer R1.1, R11.1, R13.1, R15.1, R17.1, R19.1, R26.1, R28.1, R3.1, R30.1, R37.1, R39.1, R5.1, R7.1, R9.1
- net N$10: now also U2.4; no longer U8.4
- net N$100: now also JP12.1, U8.1; no longer J14.P2, U5.1
- net N$102: now also JP13.1, U9.1; no longer J15.P2, U4.1
- net N$104: now also JP14.1, U10.1; no longer J16.P2, U6.1
- net N$107: now also U12.4; no longer U15.4
- net N$108: now also U12.3; no longer U15.3
- net N$109: now also U12.2; no longer U15.2
- net N$11: now also U2.3; no longer U8.3
- net N$111: now also U13.4; no longer U12.4
- net N$112: now also U13.3; no longer U12.3
- net N$113: now also U13.2; no longer U12.2
- net N$115: now also U14.4; no longer U11.4
- net N$116: now also U14.3; no longer U11.3
- net N$117: now also U14.2; no longer U11.2
- net N$119: now also U15.4; no longer U13.4
- net N$12: now also U2.2; no longer U8.2
- net N$120: now also U15.3; no longer U13.3
- net N$121: now also U15.2; no longer U13.2
- net N$123: now also JP9.1, U5.1; no longer J6.P2, U3.1
- net N$125: now also U11.4; no longer U14.4
- net N$126: now also U11.3; no longer U14.3
- net N$127: now also U11.2; no longer U14.2
- net N$128: now also U2.7; no longer U8.7
- net N$129: now also U11.14; no longer U14.14
- net N$13: now also U1.14; no longer U7.14
- net N$130: now also U11.13; no longer U14.13
- net N$131: now also U11.11; no longer U14.11
- net N$132: now also U11.12; no longer U14.12
- net N$133: now also U12.12; no longer U15.12
- net N$134: now also U12.14; no longer U15.14
- net N$135: now also U12.13; no longer U15.13
- net N$136: now also U12.11; no longer U15.11
- net N$137: now also U13.14; no longer U12.14
- net N$138: now also U13.13; no longer U12.13
- net N$139: now also U13.11; no longer U12.11
- net N$14: now also U1.13; no longer U7.13
- net N$140: now also U13.12; no longer U12.12
- net N$141: now also U14.14; no longer U11.14
- net N$142: now also U14.13; no longer U11.13
- net N$143: now also U14.11; no longer U11.11
- net N$144: now also U14.12; no longer U11.12
- net N$145: now also U15.12; no longer U13.12
- net N$146: now also U15.11; no longer U13.11
- net N$147: now also U15.13; no longer U13.13
- net N$148: now also U15.14; no longer U13.14
- net N$149: now also U2.8; no longer U8.8
- net N$15: now also U1.11; no longer U7.11
- net N$150: now also JP15.1, U11.1; no longer J7.P2, U14.1
- net N$152: now also JP17.1, U12.1; no longer J8.P2, U15.1
- net N$154: now also JP18.1, U13.1; no longer J9.P2, U12.1
- net N$156: now also JP19.1, U14.1; no longer J10.P2, U11.1
- net N$158: now also JP20.1, U15.1; no longer J11.P2, U13.1
- net N$16: now also U1.12; no longer U7.12
- net N$160: now also U3.5, U3.6; no longer U2.6
- net N$161: now also U3.7; no longer U2.7
- net N$162: now also U3.8; no longer U2.8
- net N$163: now also U4.5, U4.6; no longer U1.6
- net N$164: now also U4.7; no longer U1.7
- net N$165: now also U4.8; no longer U1.8
- net N$166: now also U5.5, U5.6; no longer U3.6
- net N$167: now also U5.7; no longer U3.7
- net N$168: now also U5.8; no longer U3.8
- net N$169: now also U10.8; no longer U6.8
- net N$17: now also U2.12; no longer U8.12
- net N$170: now also U10.7; no longer U6.7
- net N$171: now also U10.5, U10.6; no longer U6.6
- net N$172: now also U9.8; no longer U4.8
- net N$173: now also U9.7; no longer U4.7
- net N$174: now also U9.5, U9.6; no longer U4.6
- net N$175: now also U8.8; no longer U5.8
- net N$176: now also U8.7; no longer U5.7
- net N$177: now also U8.5, U8.6; no longer U5.6
- net N$178: now also U7.8; no longer U10.8
- net N$179: now also U7.7; no longer U10.7
- net N$18: now also U1.4; no longer U7.4
- net N$180: now also U7.5, U7.6; no longer U10.6
- net N$181: now also U6.8; no longer U9.8
- net N$182: now also U6.7; no longer U9.7
- net N$183: now also U6.5, U6.6; no longer U9.6
- net N$184: now also U15.8; no longer U13.8
- net N$186: now also U15.7; no longer U13.7
- net N$187: now also U15.5, U15.6; no longer U13.6
- net N$188: now also U14.8; no longer U11.8
- net N$189: now also U14.7; no longer U11.7
- net N$19: now also U1.3; no longer U7.3
- net N$190: now also U14.5, U14.6; no longer U11.6
- net N$191: now also U13.8; no longer U12.8
- net N$192: now also U13.7; no longer U12.7
- net N$193: now also U13.5, U13.6; no longer U12.6
- net N$194: now also U12.8; no longer U15.8
- net N$195: now also U12.7; no longer U15.7
- net N$196: now also U12.5, U12.6; no longer U15.6
- net N$197: now also U11.8; no longer U14.8
- net N$198: now also U11.7; no longer U14.7
- net N$199: now also U11.5, U11.6; no longer U14.6
- net N$20: now also U1.2; no longer U7.2
- net N$23: now also U3.4; no longer U2.4
- net N$24: now also U3.3; no longer U2.3
- net N$25: now also U3.2; no longer U2.2
- net N$27: now also U4.4; no longer U1.4
- net N$28: now also U4.3; no longer U1.3
- net N$29: now also U4.2; no longer U1.2
- net N$3: now also JP5.1, U1.1; no longer J2.P2, U7.1
- net N$31: now also U5.4; no longer U3.4
- net N$32: now also U5.3; no longer U3.3
- net N$33: now also U5.2; no longer U3.2
- net N$34: now also JP6.1, U2.1; no longer J3.P2, U8.1
- net N$36: now also JP7.1, U3.1; no longer J4.P2, U2.1
- net N$38: now also U1.7; no longer U7.7
- net N$39: now also U2.14; no longer U8.14
- net N$4: now also U1.5, U1.6; no longer U7.6
- net N$40: now also U2.13; no longer U8.13
- net N$41: now also U2.11; no longer U8.11
- net N$42: now also U3.14; no longer U2.14
- net N$43: now also U3.13; no longer U2.13
- net N$44: now also U3.11; no longer U2.11
- net N$45: now also U3.12; no longer U2.12
- net N$46: now also U4.14; no longer U1.14
- net N$47: now also U4.13; no longer U1.13
- net N$48: now also U4.11; no longer U1.11
- net N$49: now also U4.12; no longer U1.12
- net N$50: now also U5.12; no longer U3.12
- net N$51: now also U5.11; no longer U3.11
- net N$52: now also U5.13; no longer U3.13
- net N$53: now also U5.14; no longer U3.14
- net N$54: now also JP8.1, U4.1; no longer J5.P2, U1.1
- net N$55: now also U7.2; no longer U10.2
- net N$57: now also U8.4; no longer U5.4
- net N$58: now also U8.3; no longer U5.3
- net N$59: now also U8.2; no longer U5.2
- net N$6: now also U7.4; no longer U10.4
- net N$61: now also U9.4; no longer U4.4
- net N$62: now also U9.3; no longer U4.3
- net N$63: now also U9.2; no longer U4.2
- net N$65: now also U10.4; no longer U6.4
- net N$66: now also U10.3; no longer U6.3
- net N$67: now also U10.2; no longer U6.2
- net N$69: now also U6.4; no longer U9.4
- net N$7: now also U7.3; no longer U10.3
- net N$70: now also U6.3; no longer U9.3
- net N$71: now also U6.2; no longer U9.2
- net N$72: now also U1.8; no longer U7.8
- net N$73: now also U6.14; no longer U9.14
- net N$74: now also U6.13; no longer U9.13
- net N$75: now also U6.11; no longer U9.11
- net N$76: now also U6.12; no longer U9.12
- net N$77: now also U7.12; no longer U10.12
- net N$78: now also U7.14; no longer U10.14
- net N$79: now also U7.13; no longer U10.13
- net N$82: now also U7.11; no longer U10.11
- net N$83: now also U8.14; no longer U5.14
- net N$84: now also U8.13; no longer U5.13
- net N$85: now also U8.11; no longer U5.11
- net N$86: now also U8.12; no longer U5.12
- net N$87: now also U9.14; no longer U4.14
- net N$88: now also U9.13; no longer U4.13
- net N$89: now also U9.11; no longer U4.11
- net N$90: now also U9.12; no longer U4.12
- net N$91: now also U10.12; no longer U6.12
- net N$92: now also U10.11; no longer U6.11
- net N$93: now also U10.13; no longer U6.13
- net N$94: now also U10.14; no longer U6.14
- net N$95: now also U2.5, U2.6; no longer U8.6
- net N$96: now also JP10.1, U6.1; no longer J12.P2, U9.1
- net N$98: now also JP11.1, U7.1; no longer J13.P2, U10.1
Routing:
- net N$136: track 150.1 -> 529.9 mm
- net N$191: track 25.0 -> 359.9 mm
- net N$195: track 53.5 -> 325.8 mm, vias 0 -> 3
- net N$197: track 37.2 -> 294.8 mm, vias 0 -> 5
- net N$198: track 37.1 -> 289.9 mm, vias 0 -> 2
- net N$138: track 87.2 -> 311.5 mm, vias 3 -> 17
- net N$153: track 221.7 -> 0.00 mm, vias 7 -> 0
- net N$29: track 306.4 -> 89.5 mm, vias 6 -> 3
- net N$193: track 25.7 -> 238.7 mm, vias 0 -> 4
- net N$196: track 55.5 -> 267.4 mm, vias 0 -> 11
- net N$66: track 101.5 -> 310.1 mm, vias 0 -> 10
- net N$192: track 36.1 -> 244.0 mm, vias 0 -> 1
- net N$194: track 56.8 -> 261.7 mm, vias 0 -> 3
- net N$19: track 268.2 -> 65.4 mm, vias 6 -> 0
- net N$189: track 38.7 -> 239.6 mm, vias 0 -> 6
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Other:
- board size 210.3 x 100.2 mm -> 242.3 x 100.2 mm

Commit message: Added finishing touches
Parts:
- removed A1: A000067, A000067:ARDUINO_A000067
- moved U$1 6.58 mm to (156.5, 29.3)
- moved U$2 6.58 mm to (166.7, 29.3)
- moved U$3 6.58 mm to (177.0, 29.2)
- moved U$4 6.58 mm to (187.3, 29.3)
- moved U$5 6.58 mm to (197.6, 29.3)
- moved U$11 3.88 mm to (156.5, 7.20)
- moved U$12 3.88 mm to (166.7, 7.20)
- moved U$13 3.88 mm to (177.1, 7.20)
- moved U$14 3.88 mm to (187.5, 7.20)
- moved U$15 3.88 mm to (197.8, 7.20)
- moved U$10 1.46 mm to (197.9, 18.1)
- moved U$6 1.46 mm to (156.8, 18.1)
- moved U$7 1.46 mm to (167.0, 18.1)
- moved U$8 1.46 mm to (177.3, 18.1)
- moved U$9 1.46 mm to (187.7, 18.1)
Routing:
- net N$136: track 529.9 -> 81.6 mm, vias 6 -> 1
- net N$138: track 311.5 -> 83.3 mm, vias 17 -> 0
- net N$66: track 310.1 -> 143.0 mm, vias 10 -> 7
- net N$104: track 275.5 -> 120.8 mm, vias 10 -> 2
- net N$67: track 247.5 -> 100.1 mm, vias 10 -> 8
- net N$182: track 103.9 -> 250.7 mm, vias 5 -> 4
- net N$45: track 237.1 -> 95.4 mm, vias 12 -> 0
- net N$143: track 184.0 -> 63.9 mm, vias 9 -> 1
- net N$65: track 249.8 -> 131.3 mm, vias 7 -> 10
- net N$135: track 202.6 -> 85.6 mm, vias 15 -> 1
- net N$196: track 267.4 -> 160.5 mm, vias 11 -> 8
- net N$192: track 244.0 -> 350.5 mm, vias 1 -> 3
- net N$53: track 189.0 -> 84.0 mm, vias 7 -> 2
- net N$84: track 184.8 -> 86.2 mm, vias 6 -> 5
- net N$129: track 211.3 -> 118.4 mm, vias 2 -> 6
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
Commit message: Updated trace widths
Parts:
- moved SW15 185.4 mm to (226.8, 81.5)
- moved JP20 180.3 mm to (220.5, 85.2), turned to 0 degrees
- moved SW14 179.0 mm to (209.8, 81.5)
- moved R20 177.2 mm to (220.7, 79.7), turned to 270 degrees
- moved SW13 173.1 mm to (193.3, 81.1)
- moved R18 170.4 mm to (203.2, 80.2), turned to 270 degrees
- moved JP19 169.3 mm to (203.5, 85.2), turned to 0 degrees
- moved R16 164.1 mm to (186.4, 80.2), turned to 270 degrees
- moved SW12 164.1 mm to (173.6, 80.9)
- moved JP18 158.8 mm to (187.0, 85.0), turned to 0 degrees
- moved SW11 157.5 mm to (156.4, 81.1)
- moved R14 155.0 mm to (167.1, 80.1), turned to 270 degrees
- moved R12 148.6 mm to (150.1, 79.7), turned to 270 degrees
- moved JP17 145.1 mm to (167.2, 84.8), turned to 0 degrees
- moved R45 141.5 mm to (230.1, 66.9), turned to 180 degrees
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Routing:
- net N$191: track 357.2 -> 57.9 mm
- net N$192: track 350.5 -> 60.0 mm, vias 3 -> 2
- net N$169: track 67.1 -> 356.0 mm, vias 5 -> 6
- net N$106: track 9.69 -> 292.2 mm, vias 0 -> 5
- net N$195: track 330.4 -> 48.6 mm
- net N$194: track 323.7 -> 46.3 mm, vias 1 -> 2
- net N$198: track 305.8 -> 48.3 mm
- net N$118: track 9.65 -> 252.1 mm, vias 0 -> 3
- net N$110: track 9.74 -> 250.6 mm, vias 0 -> 3
- net N$68: track 9.20 -> 249.6 mm, vias 0 -> 1
- net N$197: track 274.3 -> 35.7 mm, vias 4 -> 1
- net N$114: track 9.48 -> 242.9 mm, vias 0 -> 5
- net N$122: track 14.3 -> 227.9 mm, vias 0 -> 9
- net N$60: track 9.15 -> 212.9 mm, vias 0 -> 8
- net N$56: track 9.37 -> 210.2 mm, vias 0 -> 8
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
Commit message: Switched to net labels instead of long wires
Connections:
- net N$1 renamed GND
- net N$2 renamed VMOT
- net N$80 renamed 5V
- removed net N$169 (its old number): J1.34, U10.8
- removed net N$170 (its old number): J1.32, U10.7
- removed net N$171 (its old number): J1.30, U10.5, U10.6
- removed net N$172 (its old number): J1.28, U9.8
- removed net N$173 (its old number): J1.26, U9.7
- removed net N$174 (its old number): J1.24, U9.5, U9.6
- removed net N$175 (its old number): J1.22, U8.8
- removed net N$177 (its old number): J1.18, U8.5, U8.6
- removed net N$178 (its old number): J1.16, U7.8
- removed net N$179: J1.14, U7.7
- removed net N$180 (its old number): J1.12, U7.5, U7.6
- removed net N$181: J1.10, U6.8
- removed net N$182: J1.8, U6.7
- removed net N$183: J1.6, U6.5, U6.6
- new net N$1: J1.6, U10.8
- new net N$155: J1.18, U8.8
- new net N$159: J1.22, U8.5, U8.6
- new net N$160: J1.24, U7.8
- new net N$161: J1.26, U7.7
- new net N$162: J1.28, U7.5, U7.6
- new net N$163: J1.30, U6.8
- new net N$164: J1.32, U6.7
- new net N$165: J1.34, U6.5, U6.6
- new net N$2: J1.8, U10.7
- new net N$38: J1.12, U9.8
- new net N$4: J1.10, U10.5, U10.6
- new net N$72: J1.14, U9.7
- new net N$80: J1.16, U9.5, U9.6
Routing:
- net N$169 (its old number): track 356.0 -> 0.00 mm, vias 6 -> 0
- net N$183: track 289.8 -> 0.00 mm, vias 11 -> 0
- net N$165: track 0.00 -> 258.9 mm, vias 0 -> 10
- net N$182: track 245.2 -> 0.00 mm, vias 11 -> 0
- net N$179: track 241.5 -> 0.00 mm, vias 12 -> 0
- net N$159: track 0.00 -> 229.2 mm, vias 0 -> 12
- net N$160: track 0.00 -> 201.9 mm, vias 0 -> 7
- net N$123: track 72.6 -> 273.2 mm, vias 5 -> 9
- net N$164: track 0.00 -> 197.0 mm, vias 0 -> 11
- net N$178 (its old number): track 193.3 -> 0.00 mm, vias 10 -> 0
- net N$161: track 0.00 -> 185.0 mm, vias 0 -> 5
- net N$122: track 227.9 -> 402.5 mm, vias 9 -> 5
- net N$163: track 0.00 -> 171.6 mm, vias 0 -> 4
- net N$124: track 97.3 -> 261.3 mm, vias 6 -> 13
- net N$80: track 0.00 -> 161.8 mm, vias 0 -> 6
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