File: StepperBoard/StepperBoard.sch (EAGLE design)
At the start: 129 parts, among them J1 F-2X18-DIL-100, U1 A4988_STEPPER_MOTOR_DRIVER_CA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, U10 A4988_STEPPER_MOTOR_DRIVER_CA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, U11 A4988_STEPPER_MOTOR_DRIVER_CA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, U12 A4988_STEPPER_MOTOR_DRIVER_CA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, U13 A4988_STEPPER_MOTOR_DRIVER_CA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, U14 A4988_STEPPER_MOTOR_DRIVER_CA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, U15 A4988_STEPPER_MOTOR_DRIVER_CA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, U2 A4988_STEPPER_MOTOR_DRIVER_CA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, U3 A4988_STEPPER_MOTOR_DRIVER_CA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, U4 A4988_STEPPER_MOTOR_DRIVER_CA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, U5 A4988_STEPPER_MOTOR_DRIVER_CA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, U6 A4988_STEPPER_MOTOR_DRIVER_CA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, U7 A4988_STEPPER_MOTOR_DRIVER_CA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, U8 A4988_STEPPER_MOTOR_DRIVER_CA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, U9 A4988_STEPPER_MOTOR_DRIVER_CA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

Commit message: Add files via upload
Board design updated
Parts:
- removed J10, J11, J12, J13, J14, J15, J16, J2, J3, J4, J5, J6, J7, J8, J9: (no value), SparkFun-Connectors:CONN_022.54MM_SCREWTERM
- removed R1, R11, R13, R15, R17, R19, R26, R28, R3, R30, R37, R39, R5, R7, R9: 4.7k, SparkFun-Resistors:4.7KOHM-0603-1/10W-1%
- added JP10, JP11, JP12, JP13, JP14, JP15, JP17, JP18, JP19, JP20, JP5, JP6, JP7, JP8, JP9: (no value), pinhead:PINHD-1X1
Connections:
- removed net N$101: J14.1, R15.2, U5.!RESET
- removed net N$103: J15.1, R17.2, U4.!RESET
- removed net N$105: J16.1, R19.2, U6.!RESET
- removed net N$124: J6.1, R9.2, U3.!RESET
- removed net N$151: J7.1, R26.2, U14.!RESET
- removed net N$153: J8.1, R28.2, U15.!RESET
- removed net N$155: J9.1, R30.2, U12.!RESET
- removed net N$157: J10.1, R37.2, U11.!RESET
- removed net N$159: J11.1, R39.2, U13.!RESET
- removed net N$35: J3.1, R3.2, U8.!RESET
- removed net N$37: J4.1, R5.2, U2.!RESET
- removed net N$8: J2.1, R1.2, U7.!RESET
- removed net N$81: J5.1, R7.2, U1.!RESET
- removed net N$97: J12.1, R11.2, U9.!RESET
- removed net N$99: J13.1, R13.2, U10.!RESET
- net N$1: no longer R1.1, R11.1, R13.1, R15.1, R17.1, R19.1, R26.1, R28.1, R3.1, R30.1, R37.1, R39.1, R5.1, R7.1, R9.1
- net N$10: now also U2.MS3; no longer U8.MS3
- net N$100: now also JP12.1, U8.!ENABLE; no longer J14.2, U5.!ENABLE
- net N$102: now also JP13.1, U9.!ENABLE; no longer J15.2, U4.!ENABLE
- net N$104: now also JP14.1, U10.!ENABLE; no longer J16.2, U6.!ENABLE
- net N$107: now also U12.MS3; no longer U15.MS3
- net N$108: now also U12.MS2; no longer U15.MS2
- net N$109: now also U12.MS1; no longer U15.MS1
- net N$11: now also U2.MS2; no longer U8.MS2
- net N$111: now also U13.MS3; no longer U12.MS3
- net N$112: now also U13.MS2; no longer U12.MS2
- net N$113: now also U13.MS1; no longer U12.MS1
- net N$115: now also U14.MS3; no longer U11.MS3
- net N$116: now also U14.MS2; no longer U11.MS2
- net N$117: now also U14.MS1; no longer U11.MS1
- net N$119: now also U15.MS3; no longer U13.MS3
- net N$12: now also U2.MS1; no longer U8.MS1
- net N$120: now also U15.MS2; no longer U13.MS2
- net N$121: now also U15.MS1; no longer U13.MS1
- net N$123: now also JP9.1, U5.!ENABLE; no longer J6.2, U3.!ENABLE
- net N$125: now also U11.MS3; no longer U14.MS3
- net N$126: now also U11.MS2; no longer U14.MS2
- net N$127: now also U11.MS1; no longer U14.MS1
- net N$128: now also U2.STEP; no longer U8.STEP
- net N$129: now also U11.2B; no longer U14.2B
- net N$13: now also U1.2B; no longer U7.2B
- net N$130: now also U11.2A; no longer U14.2A
- net N$131: now also U11.1B; no longer U14.1B
- net N$132: now also U11.1A; no longer U14.1A
- net N$133: now also U12.1A; no longer U15.1A
- net N$134: now also U12.2B; no longer U15.2B
- net N$135: now also U12.2A; no longer U15.2A
- net N$136: now also U12.1B; no longer U15.1B
- net N$137: now also U13.2B; no longer U12.2B
- net N$138: now also U13.2A; no longer U12.2A
- net N$139: now also U13.1B; no longer U12.1B
- net N$14: now also U1.2A; no longer U7.2A
- net N$140: now also U13.1A; no longer U12.1A
- net N$141: now also U14.2B; no longer U11.2B
- net N$142: now also U14.2A; no longer U11.2A
- net N$143: now also U14.1B; no longer U11.1B
- net N$144: now also U14.1A; no longer U11.1A
- net N$145: now also U15.1A; no longer U13.1A
- net N$146: now also U15.1B; no longer U13.1B
- net N$147: now also U15.2A; no longer U13.2A
- net N$148: now also U15.2B; no longer U13.2B
- net N$149: now also U2.DIR; no longer U8.DIR
- net N$15: now also U1.1B; no longer U7.1B
- net N$150: now also JP15.1, U11.!ENABLE; no longer J7.2, U14.!ENABLE
- net N$152: now also JP17.1, U12.!ENABLE; no longer J8.2, U15.!ENABLE
- net N$154: now also JP18.1, U13.!ENABLE; no longer J9.2, U12.!ENABLE
- net N$156: now also JP19.1, U14.!ENABLE; no longer J10.2, U11.!ENABLE
- net N$158: now also JP20.1, U15.!ENABLE; no longer J11.2, U13.!ENABLE
- net N$16: now also U1.1A; no longer U7.1A
- net N$160: now also U3.!RESET, U3.!SLEEP; no longer U2.!SLEEP
- net N$161: now also U3.STEP; no longer U2.STEP
- net N$162: now also U3.DIR; no longer U2.DIR
- net N$163: now also U4.!RESET, U4.!SLEEP; no longer U1.!SLEEP
- net N$164: now also U4.STEP; no longer U1.STEP
- net N$165: now also U4.DIR; no longer U1.DIR
- net N$166: now also U5.!RESET, U5.!SLEEP; no longer U3.!SLEEP
- net N$167: now also U5.STEP; no longer U3.STEP
- net N$168: now also U5.DIR; no longer U3.DIR
- net N$169: now also U10.DIR; no longer U6.DIR
- net N$17: now also U2.1A; no longer U8.1A
- net N$170: now also U10.STEP; no longer U6.STEP
- net N$171: now also U10.!RESET, U10.!SLEEP; no longer U6.!SLEEP
- net N$172: now also U9.DIR; no longer U4.DIR
- net N$173: now also U9.STEP; no longer U4.STEP
- net N$174: now also U9.!RESET, U9.!SLEEP; no longer U4.!SLEEP
- net N$175: now also U8.DIR; no longer U5.DIR
- net N$176: now also U8.STEP; no longer U5.STEP
- net N$177: now also U8.!RESET, U8.!SLEEP; no longer U5.!SLEEP
- net N$178: now also U7.DIR; no longer U10.DIR
- net N$179: now also U7.STEP; no longer U10.STEP
- net N$18: now also U1.MS3; no longer U7.MS3
- net N$180: now also U7.!RESET, U7.!SLEEP; no longer U10.!SLEEP
- net N$181: now also U6.DIR; no longer U9.DIR
- net N$182: now also U6.STEP; no longer U9.STEP
- net N$183: now also U6.!RESET, U6.!SLEEP; no longer U9.!SLEEP
- net N$184: now also U15.DIR; no longer U13.DIR
- net N$186: now also U15.STEP; no longer U13.STEP
- net N$187: now also U15.!RESET, U15.!SLEEP; no longer U13.!SLEEP
- net N$188: now also U14.DIR; no longer U11.DIR
- net N$189: now also U14.STEP; no longer U11.STEP
- net N$19: now also U1.MS2; no longer U7.MS2
- net N$190: now also U14.!RESET, U14.!SLEEP; no longer U11.!SLEEP
- net N$191: now also U13.DIR; no longer U12.DIR
- net N$192: now also U13.STEP; no longer U12.STEP
- net N$193: now also U13.!RESET, U13.!SLEEP; no longer U12.!SLEEP
- net N$194: now also U12.DIR; no longer U15.DIR
- net N$195: now also U12.STEP; no longer U15.STEP
- net N$196: now also U12.!RESET, U12.!SLEEP; no longer U15.!SLEEP
- net N$197: now also U11.DIR; no longer U14.DIR
- net N$198: now also U11.STEP; no longer U14.STEP
- net N$199: now also U11.!RESET, U11.!SLEEP; no longer U14.!SLEEP
- net N$20: now also U1.MS1; no longer U7.MS1
- net N$23: now also U3.MS3; no longer U2.MS3
- net N$24: now also U3.MS2; no longer U2.MS2
- net N$25: now also U3.MS1; no longer U2.MS1
- net N$27: now also U4.MS3; no longer U1.MS3
- net N$28: now also U4.MS2; no longer U1.MS2
- net N$29: now also U4.MS1; no longer U1.MS1
- net N$3: now also JP5.1, U1.!ENABLE; no longer J2.2, U7.!ENABLE
- net N$31: now also U5.MS3; no longer U3.MS3
- net N$32: now also U5.MS2; no longer U3.MS2
- net N$33: now also U5.MS1; no longer U3.MS1
- net N$34: now also JP6.1, U2.!ENABLE; no longer J3.2, U8.!ENABLE
- net N$36: now also JP7.1, U3.!ENABLE; no longer J4.2, U2.!ENABLE
- net N$38: now also U1.STEP; no longer U7.STEP
- net N$39: now also U2.2B; no longer U8.2B
- net N$4: now also U1.!RESET, U1.!SLEEP; no longer U7.!SLEEP
- net N$40: now also U2.2A; no longer U8.2A
- net N$41: now also U2.1B; no longer U8.1B
- net N$42: now also U3.2B; no longer U2.2B
- net N$43: now also U3.2A; no longer U2.2A
- net N$44: now also U3.1B; no longer U2.1B
- net N$45: now also U3.1A; no longer U2.1A
- net N$46: now also U4.2B; no longer U1.2B
- net N$47: now also U4.2A; no longer U1.2A
- net N$48: now also U4.1B; no longer U1.1B
- net N$49: now also U4.1A; no longer U1.1A
- net N$50: now also U5.1A; no longer U3.1A
- net N$51: now also U5.1B; no longer U3.1B
- net N$52: now also U5.2A; no longer U3.2A
- net N$53: now also U5.2B; no longer U3.2B
- net N$54: now also JP8.1, U4.!ENABLE; no longer J5.2, U1.!ENABLE
- net N$55: now also U7.MS1; no longer U10.MS1
- net N$57: now also U8.MS3; no longer U5.MS3
- net N$58: now also U8.MS2; no longer U5.MS2
- net N$59: now also U8.MS1; no longer U5.MS1
- net N$6: now also U7.MS3; no longer U10.MS3
- net N$61: now also U9.MS3; no longer U4.MS3
- net N$62: now also U9.MS2; no longer U4.MS2
- net N$63: now also U9.MS1; no longer U4.MS1
- net N$65: now also U10.MS3; no longer U6.MS3
- net N$66: now also U10.MS2; no longer U6.MS2
- net N$67: now also U10.MS1; no longer U6.MS1
- net N$69: now also U6.MS3; no longer U9.MS3
- net N$7: now also U7.MS2; no longer U10.MS2
- net N$70: now also U6.MS2; no longer U9.MS2
- net N$71: now also U6.MS1; no longer U9.MS1
- net N$72: now also U1.DIR; no longer U7.DIR
- net N$73: now also U6.2B; no longer U9.2B
- net N$74: now also U6.2A; no longer U9.2A
- net N$75: now also U6.1B; no longer U9.1B
- net N$76: now also U6.1A; no longer U9.1A
- net N$77: now also U7.1A; no longer U10.1A
- net N$78: now also U7.2B; no longer U10.2B
- net N$79: now also U7.2A; no longer U10.2A
- net N$82: now also U7.1B; no longer U10.1B
- net N$83: now also U8.2B; no longer U5.2B
- net N$84: now also U8.2A; no longer U5.2A
- net N$85: now also U8.1B; no longer U5.1B
- net N$86: now also U8.1A; no longer U5.1A
- net N$87: now also U9.2B; no longer U4.2B
- net N$88: now also U9.2A; no longer U4.2A
- net N$89: now also U9.1B; no longer U4.1B
- net N$90: now also U9.1A; no longer U4.1A
- net N$91: now also U10.1A; no longer U6.1A
- net N$92: now also U10.1B; no longer U6.1B
- net N$93: now also U10.2A; no longer U6.2A
- net N$94: now also U10.2B; no longer U6.2B
- net N$95: now also U2.!RESET, U2.!SLEEP; no longer U8.!SLEEP
- net N$96: now also JP10.1, U6.!ENABLE; no longer J12.2, U9.!ENABLE
- net N$98: now also JP11.1, U7.!ENABLE; no longer J13.2, U10.!ENABLE
Other:
- moved on the sheet: U1, U10, U11, U12, U13, U14, U15, U2, U3, U4, U5, U6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

Commit message: Added finishing touches
Parts:
- removed A1: A000067, A000067:A000067
Changed lines of the file:
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@@
 <part name="J1" library="con-headers-jp" deviceset="F-2X18-" device="DIL-100"/>
 <part name="JP16" library="pinhead" library_urn="urn:adsk.eagle:library:325" deviceset="PINHD-1X8" device="" package3d_urn="urn:adsk.eagle:package:22409/2"/>
-<part name="A1" library="A000067" deviceset="A000067" device=""/>
 <part name="R21" library="SparkFun-Resistors" deviceset="4.7KOHM" device="-0603-1/10W-1%" value="4.7k"/>
 <part name="R22" library="SparkFun-Resistors" deviceset="4.7KOHM" device="-0603-1/10W-1%" value="4.7k"/>
@@
 <attribute name="VALUE" x="643.89" y="454.66" size="1.778" layer="96" rot="R180"/>
 </instance>
-<instance part="A1" gate="G$1" x="1031.24" y="393.7" smashed="yes">
-<attribute name="NAME" x="1016" y="455.295" size="1.778" layer="95"/>
-<attribute name="VALUE" x="1016" y="330.2" size="1.778" layer="96"/>
-</instance>
 <instance part="R21" gate="G$1" x="185.42" y="358.14" smashed="yes">

Commit message: Switched to net labels instead of long wires
Connections:
- net N$1 renamed GND
- net N$2 renamed VMOT
- net N$80 renamed 5V
- removed net N$169 (its old number): J1.34, U10.DIR
- removed net N$170 (its old number): J1.32, U10.STEP
- removed net N$171 (its old number): J1.30, U10.!RESET, U10.!SLEEP
- removed net N$172 (its old number): J1.28, U9.DIR
- removed net N$173 (its old number): J1.26, U9.STEP
- removed net N$174 (its old number): J1.24, U9.!RESET, U9.!SLEEP
- removed net N$175 (its old number): J1.22, U8.DIR
- removed net N$177 (its old number): J1.18, U8.!RESET, U8.!SLEEP
- removed net N$178 (its old number): J1.16, U7.DIR
- removed net N$179: J1.14, U7.STEP
- removed net N$180 (its old number): J1.12, U7.!RESET, U7.!SLEEP
- removed net N$181: J1.10, U6.DIR
- removed net N$182: J1.8, U6.STEP
- removed net N$183: J1.6, U6.!RESET, U6.!SLEEP
- new net N$1: J1.6, U10.DIR
- new net N$155: J1.18, U8.DIR
- new net N$159: J1.22, U8.!RESET, U8.!SLEEP
- new net N$160: J1.24, U7.DIR
- new net N$161: J1.26, U7.STEP
- new net N$162: J1.28, U7.!RESET, U7.!SLEEP
- new net N$163: J1.30, U6.DIR
- new net N$164: J1.32, U6.STEP
- new net N$165: J1.34, U6.!RESET, U6.!SLEEP
- new net N$2: J1.8, U10.STEP
- new net N$38: J1.12, U9.DIR
- new net N$4: J1.10, U10.!RESET, U10.!SLEEP
- new net N$72: J1.14, U9.STEP
- new net N$80: J1.16, U9.!RESET, U9.!SLEEP
Other:
- moved on the sheet: C1, C10, C11, C12, C13, C14, C15, C2, C3, C4, C5, C6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
