File: StepperBoard_v2/v2.brd (EAGLE design)
At the start: 302.4 x 100.1 mm, 69 parts, among them IC1 2969-MP6500, IC10 2969-MP6500, IC11 2969-MP6500, IC12 2969-MP6500, IC13 2969-MP6500, IC14 2969-MP6500, IC15 2969-MP6500, IC2 2969-MP6500, IC3 2969-MP6500, IC4 2969-MP6500, IC5 2969-MP6500, IC6 2969-MP6500, IC7 2969-MP6500, IC8 2969-MP6500, IC9 2969-MP6500, J1 F-2X18-DIL-100

Commit message: Made recommended changes
Parts:
- added R1, R10, R11, R12, R13, R14, R15, R2, R3, R4, R5, R6, R7, R8, R9: 2.0k, SparkFun-Resistors:0603
- moved X2 266.7 mm to (26.4, 89.9), turned to 0 degrees
- moved U$16 256.3 mm to (28.1, 68.5), turned to 0 degrees
- moved JP2 243.5 mm to (34.4, 20.2), turned to 0 degrees
- moved SV6 229.4 mm to (251.2, 71.4)
- moved SV15 216.9 mm to (250.6, 23.5)
- moved JP4 209.1 mm to (52.2, 68.5), turned to 0 degrees
- moved SV5 207.1 mm to (223.2, 71.8)
- moved JP16 198.9 mm to (57.3, 20.2), turned to 0 degrees
- moved SV14 186.9 mm to (223.5, 23.5)
- moved C6 183.4 mm to (264.8, 72.9), turned to 0 degrees
- moved SV4 179.1 mm to (195.4, 71.5)
- moved IC6 177.2 mm to (264.9, 68.0), turned to 0 degrees
- moved C5 174.8 mm to (237.2, 73.2), turned to 0 degrees
- moved F1 173.6 mm to (62.6, 90.3), turned to 0 degrees
- moved IC5 170.2 mm to (237.2, 68.1), turned to 0 degrees
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Connections:
- net 5V: now also R1.1, R10.1, R11.1, R12.1, R13.1, R14.1, R15.1, R2.1, R3.1, R4.1, R5.1, R6.1, R7.1, R8.1, R9.1; no longer SV1.2, SV1.4, SV10.2, SV10.4, SV11.2, SV11.4, SV12.2, SV12.4, SV13.2, SV13.4, SV14.2, SV14.4, SV15.2, SV15.4, SV2.2, SV2.4, SV3.2, SV3.4, SV4.2, SV4.4, SV5.2, SV5.4, SV6.2, SV6.4, SV7.2, SV7.4, SV8.2, SV8.4, SV9.2, SV9.4
- net GND: now also SV1.2, SV1.4, SV10.2, SV10.4, SV11.2, SV11.4, SV12.2, SV12.4, SV13.2, SV13.4, SV14.2, SV14.4, SV15.2, SV15.4, SV2.2, SV2.4, SV3.2, SV3.4, SV4.2, SV4.4, SV5.2, SV5.4, SV6.2, SV6.4, SV7.2, SV7.4, SV8.2, SV8.4, SV9.2, SV9.4
- net N$1: now also R15.2
- net N$101: now also R10.2
- net N$104: now also R11.2
- net N$15: now also R1.2
- net N$20: now also R2.2
- net N$27: now also R3.2
- net N$42: now also R4.2
- net N$49: now also R5.2
- net N$56: now also R6.2
- net N$71: now also R14.2
- net N$78: now also R13.2
- net N$85: now also R12.2
- net N$92: now also R7.2
- net N$95: now also R8.2
- net N$98: now also R9.2
Routing:
- net 5V: track 510.2 -> 787.7 mm, vias 0 -> 8
- net GND: track 696.9 -> 928.8 mm, vias 2 -> 16
- net N$15: track 245.2 -> 57.1 mm, vias 2 -> 1
- net N$37: track 90.8 -> 263.9 mm, vias 2 -> 3
- net N$31: track 93.6 -> 240.0 mm, vias 4 -> 2
- net N$33: track 104.7 -> 246.8 mm
- net N$14: track 178.1 -> 50.8 mm, vias 5 -> 1
- net N$57: track 151.4 -> 277.0 mm
- net N$58: track 151.0 -> 276.3 mm, vias 1 -> 0
- net N$92: track 155.8 -> 31.4 mm, vias 3 -> 2
- net N$93: track 153.8 -> 31.8 mm, vias 3 -> 0
- net N$13: track 171.4 -> 50.0 mm, vias 3 -> 1
- net N$105: track 107.4 -> 225.4 mm
- net N$95: track 182.9 -> 65.8 mm, vias 2 -> 3
- net N$94: track 140.8 -> 27.0 mm, vias 3 -> 0
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
Commit message: Design is ready for order
Parts:
- removed JP16: (no value), pinhead:1X08
- removed U$16: PINHD-1X10, adafruit:1X10-BIG
- removed X2: (no value), con-wago-500:W237-4
- added CR1, CR10, CR11, CR12, CR13, CR14, CR15, CR2, CR3, CR4, CR5, CR6, CR7, CR8, CR9: PESD2CAN24DBZRQ1, TVS_Diode:SOT-23_DBZ_TEX
- added F10, F11, F12, F13, F14, F15, F2, F3, F4, F5, F6, F7, F8, F9: (no value), Fuse:0154SERIES_LTF
- J1: value F-2X18-DIL-100 -> 1888700; device con-headers-jp:DIL-100-2X18 -> PheonixContactTerm:CONN_1888700_PXC
- JP2: device pinhead:1X08 -> pinhead:2X18
- moved R6 134.9 mm to (116.9, 48.8)
- moved SV6 134.8 mm to (117.0, 57.9)
- moved IC6 134.1 mm to (131.2, 57.9)
- moved C6 134.0 mm to (131.2, 63.2)
- moved C10 133.6 mm to (252.4, 63.2)
- moved IC10 133.6 mm to (252.4, 57.9)
- moved R10 130.6 mm to (236.6, 48.8)
- moved SV10 130.1 mm to (236.6, 57.9)
- moved J1 104.8 mm to (27.3, 128.6), turned to 0 degrees
- moved F1 72.5 mm to (131.2, 113.7)
- moved JP2 70.2 mm to (92.5, 59.8), turned to 90 degrees
- moved JP1 47.9 mm to (34.0, 33.1)
- moved J2 47.6 mm to (60.9, 128.4)
- moved J3 46.2 mm to (75.5, 128.4)
- moved J4 45.0 mm to (90.0, 128.4)
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Connections:
- removed net GND: C1.-, C10.-, C11.-, C12.-, C13.-, C14.-, C15.-, C2.-, C3.-, C4.-, C5.-, C6.-, C7.-, C8.-, C9.-, IC1.15, IC1.9, IC10.15, IC10.9, IC11.15, IC11.9, IC12.15, IC12.9, IC13.15, IC13.9, IC14.15, IC14.9, IC15.15, IC15.9, IC2.15, IC2.9, IC3.15, IC3.9, IC4.15, IC4.9, IC5.15, IC5.9, IC6.15, IC6.9, IC7.15, IC7.9, IC8.15, IC8.9, IC9.15, IC9.9, SV1.2, SV1.4, SV10.2, SV10.4, SV11.2, SV11.4, SV12.2, SV12.4, SV13.2, SV13.4, SV14.2, SV14.4, SV15.2, SV15.4, SV2.2, SV2.4, SV3.2, SV3.4, SV4.2, SV4.4, SV5.2, SV5.4, SV6.2, SV6.4, SV7.2, SV7.4, SV8.2, SV8.4, SV9.2, SV9.4, X2.2, X2.3
- removed net N$1: IC11.6, JP16.8, R15.2
- removed net N$100: IC9.8, J1.24
- removed net N$101: IC10.6, J1.26, R10.2
- removed net N$102: IC10.7, J1.28
- removed net N$103: IC10.8, J1.30
- removed net N$104: IC15.6, JP1.4, R11.2
- removed net N$105: IC15.7, JP1.3
- removed net N$106: IC15.8, JP1.2
- removed net N$13: IC1.8, J1.7
- removed net N$14: IC1.7, J1.5
- removed net N$15: IC1.6, J1.3, R1.2
- removed net N$20: IC2.6, J1.9, R2.2
- removed net N$21: IC2.7, J1.11
- removed net N$22: IC2.8, J1.13
- removed net N$27: IC3.6, J1.15, R3.2
- removed net N$28: IC3.7, J1.17
- removed net N$29: IC3.8, J1.19
- removed net N$4: F1.1, X2.1
- removed net N$42: IC4.6, J1.21, R4.2
- removed net N$43: IC4.7, J1.23
- removed net N$44: IC4.8, J1.25
- removed net N$49: IC5.6, J1.27, R5.2
- removed net N$50: IC5.7, J1.29
- removed net N$51: IC5.8, J1.31
- removed net N$56: IC6.6, J1.33, R6.2
- removed net N$57: IC6.7, J1.4
- removed net N$58: IC6.8, J1.6
- removed net N$7: IC11.7, JP16.7
- removed net N$71: IC12.6, JP16.5, R14.2
- removed net N$72: IC12.7, JP16.4
- removed net N$73: IC12.8, JP16.3
- removed net N$78: IC13.6, JP16.2, R13.2
- removed net N$79: IC13.7, JP16.1
- removed net N$8: IC11.8, JP16.6
- removed net N$80: IC13.8, JP1.8
- removed net N$85: IC14.6, JP1.7, R12.2
- removed net N$86: IC14.7, JP1.6
- removed net N$87: IC14.8, JP1.5
- removed net N$92: IC7.6, J1.8, R7.2
- removed net N$93: IC7.7, J1.10
- removed net N$94: IC7.8, J1.12
- removed net N$95: IC8.6, J1.14, R8.2
- removed net N$96: IC8.7, J1.16
- removed net N$97: IC8.8, J1.18
- removed net N$98: IC9.6, J1.20, R9.2
- removed net N$99: IC9.7, J1.22
- removed net VMOT: C1.+, C10.+, C11.+, C12.+, C13.+, C14.+, C15.+, C2.+, C3.+, C4.+, C5.+, C6.+, C7.+, C8.+, C9.+, F1.2, IC1.16, IC10.16, IC11.16, IC12.16, IC13.16, IC14.16, IC15.16, IC2.16, IC3.16, IC4.16, IC5.16, IC6.16, IC7.16, IC8.16, IC9.16
- new net DIR1: IC1.8, JP2.7
- new net DIR10: IC10.8, JP2.32
- new net DIR11: IC11.8, JP3.6
- new net DIR12: IC12.8, JP3.3
- new net DIR13: IC13.8, JP4.8
- new net DIR14: IC14.8, JP4.5
- new net DIR15: IC15.8, JP4.2
- new net DIR2: IC2.8, JP2.13
- new net DIR3: IC3.8, JP2.19
- new net DIR4: IC4.8, JP2.25
- new net DIR5: IC5.8, JP2.31
- new net DIR6: IC6.8, JP2.8
- new net DIR7: IC7.8, JP2.14
- new net DIR8: IC8.8, JP2.20
- new net DIR9: IC9.8, JP2.26
- new net GND1: IC1.9, IC10.9, IC11.9, IC12.9, IC13.9, IC14.9, IC15.9, IC2.9, IC3.9, IC4.9, IC5.9, IC6.9, IC7.9, IC8.9, IC9.9, J1.2, SV1.2, SV1.4, SV10.2, SV10.4, SV11.2, SV11.4, SV12.2, SV12.4, SV13.2, SV13.4, SV14.2, SV14.4, SV15.2, SV15.4, SV2.2, SV2.4, SV3.2, SV3.4, SV4.2, SV4.4, SV5.2, SV5.4, SV6.2, SV6.4, SV7.2, SV7.4, SV8.2, SV8.4, SV9.2, SV9.4
- new net GND2: C1.-, C10.-, C11.-, C12.-, C13.-, C14.-, C15.-, C2.-, C3.-, C4.-, C5.-, C6.-, C7.-, C8.-, C9.-, CR1.3, CR10.3, CR11.3, CR12.3, CR13.3, CR14.3, CR15.3, CR2.3, CR3.3, CR4.3, CR5.3, CR6.3, CR7.3, CR8.3, CR9.3, IC1.15, IC10.15, IC11.15, IC12.15, IC13.15, IC14.15, IC15.15, IC2.15, IC3.15, IC4.15, IC5.15, IC6.15, IC7.15, IC8.15, IC9.15, J1.3
- new net N$182: F1.1, F10.1, F11.1, F12.1, F13.1, F14.1, F15.1, F2.1, F3.1, F4.1, F5.1, F6.1, F7.1, F8.1, F9.1, J1.4
- new net SLP1: IC1.6, JP2.3, R1.2
- new net SLP10: IC10.6, JP2.28, R10.2
- new net SLP11: IC11.6, JP3.8, R11.2
- new net SLP12: IC12.6, JP3.5, R12.2
- new net SLP13: IC13.6, JP3.2, R13.2
- new net SLP14: IC14.6, JP4.7, R14.2
- new net SLP15: IC15.6, JP4.4, R15.2
- new net SLP2: IC2.6, JP2.9, R2.2
- new net SLP3: IC3.6, JP2.15, R3.2
- new net SLP4: IC4.6, JP2.21, R4.2
- new net SLP5: IC5.6, JP2.27, R5.2
- new net SLP6: IC6.6, JP2.4, R6.2
- new net SLP7: IC7.6, JP2.10, R7.2
- new net SLP8: IC8.6, JP2.16, R8.2
- new net SLP9: IC9.6, JP2.22, R9.2
- new net STEP1: IC1.7, JP2.5
- new net STEP10: IC10.7, JP2.30
- new net STEP11: IC11.7, JP3.7
- new net STEP12: IC12.7, JP3.4
- new net STEP13: IC13.7, JP3.1
- new net STEP14: IC14.7, JP4.6
- new net STEP15: IC15.7, JP4.3
- new net STEP2: IC2.7, JP2.11
- new net STEP3: IC3.7, JP2.17
- new net STEP4: IC4.7, JP2.23
- new net STEP5: IC5.7, JP2.29
- new net STEP6: IC6.7, JP2.6
- new net STEP7: IC7.7, JP2.12
- new net STEP8: IC8.7, JP2.18
- new net STEP9: IC9.7, JP2.24
- new net VMOT1: C1.+, CR1.1, CR1.2, F1.2, IC1.16
- new net VMOT10: C10.+, CR10.1, CR10.2, F10.2, IC10.16
- new net VMOT11: C11.+, CR11.1, CR11.2, F11.2, IC11.16
- new net VMOT12: C12.+, CR12.1, CR12.2, F12.2, IC12.16
- new net VMOT13: C13.+, CR13.1, CR13.2, F13.2, IC13.16
- new net VMOT14: C14.+, CR14.1, CR14.2, F14.2, IC14.16
- new net VMOT15: C15.+, CR15.1, CR15.2, F15.2, IC15.16
- new net VMOT2: C2.+, CR2.1, CR2.2, F2.2, IC2.16
- new net VMOT3: C3.+, CR3.1, CR3.2, F3.2, IC3.16
- new net VMOT4: C4.+, CR4.1, CR4.2, F4.2, IC4.16
- new net VMOT5: C5.+, CR5.1, CR5.2, F5.2, IC5.16
- new net VMOT6: C6.+, CR6.1, CR6.2, F6.2, IC6.16
- new net VMOT7: C7.+, CR7.1, CR7.2, F7.2, IC7.16
- new net VMOT8: C8.+, CR8.1, CR8.2, F8.2, IC8.16
- new net VMOT9: C9.+, CR9.1, CR9.2, F9.2, IC9.16
- net 5V: now also J1.1; no longer X2.4
Routing:
- net GND: track 928.8 -> 0.00 mm, vias 16 -> 0
- net GND2: track 0.00 -> 811.9 mm, vias 0 -> 5
- net GND1: track 0.00 -> 738.2 mm, vias 0 -> 3
- net N$182: track 0.00 -> 646.9 mm, vias 0 -> 15
- net VMOT: track 597.7 -> 0.00 mm, vias 14 -> 0
- net SLP5: track 0.00 -> 356.6 mm, vias 0 -> 1
- net N$57: track 277.0 -> 0.00 mm, vias 2 -> 0
- net N$58: track 276.3 -> 0.00 mm
- net SLP10: track 0.00 -> 266.9 mm, vias 0 -> 3
- net DIR5: track 0.00 -> 266.7 mm, vias 0 -> 1
- net STEP5: track 0.00 -> 246.0 mm, vias 0 -> 2
- net DIR10: track 0.00 -> 241.3 mm, vias 0 -> 2
- net STEP9: track 0.00 -> 229.7 mm, vias 0 -> 2
- net N$56: track 226.4 -> 0.00 mm, vias 2 -> 0
- net N$105: track 225.4 -> 0.00 mm, vias 1 -> 0
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Other:
- board size 302.4 x 100.1 mm -> 295 x 145 mm
