File: StepperBoard_v2/v2.sch (EAGLE design)
At the start: 69 parts, among them IC1 2969-MP6500, IC10 2969-MP6500, IC11 2969-MP6500, IC12 2969-MP6500, IC13 2969-MP6500, IC14 2969-MP6500, IC15 2969-MP6500, IC2 2969-MP6500, IC3 2969-MP6500, IC4 2969-MP6500, IC5 2969-MP6500, IC6 2969-MP6500, IC7 2969-MP6500, IC8 2969-MP6500, IC9 2969-MP6500, J1 F-2X18-DIL-100

Commit message: Made recommended changes
Parts:
- added R1, R10, R11, R12, R13, R14, R15, R2, R3, R4, R5, R6, R7, R8, R9: 2.0k, SparkFun-Resistors:2.0KOHM-0603-1/10W-5%
Connections:
- net 5V: now also R1.1, R10.1, R11.1, R12.1, R13.1, R14.1, R15.1, R2.1, R3.1, R4.1, R5.1, R6.1, R7.1, R8.1, R9.1; no longer SV1.2, SV1.4, SV10.2, SV10.4, SV11.2, SV11.4, SV12.2, SV12.4, SV13.2, SV13.4, SV14.2, SV14.4, SV15.2, SV15.4, SV2.2, SV2.4, SV3.2, SV3.4, SV4.2, SV4.4, SV5.2, SV5.4, SV6.2, SV6.4, SV7.2, SV7.4, SV8.2, SV8.4, SV9.2, SV9.4
- net GND: now also SV1.2, SV1.4, SV10.2, SV10.4, SV11.2, SV11.4, SV12.2, SV12.4, SV13.2, SV13.4, SV14.2, SV14.4, SV15.2, SV15.4, SV2.2, SV2.4, SV3.2, SV3.4, SV4.2, SV4.4, SV5.2, SV5.4, SV6.2, SV6.4, SV7.2, SV7.4, SV8.2, SV8.4, SV9.2, SV9.4
- net N$1: now also R15.2
- net N$101: now also R10.2
- net N$104: now also R11.2
- net N$15: now also R1.2
- net N$20: now also R2.2
- net N$27: now also R3.2
- net N$42: now also R4.2
- net N$49: now also R5.2
- net N$56: now also R6.2
- net N$71: now also R14.2
- net N$78: now also R13.2
- net N$85: now also R12.2
- net N$92: now also R7.2
- net N$95: now also R8.2
- net N$98: now also R9.2
Other:
- moved on the sheet: SV10, SV13, SV15, SV3, SV5, SV9

Commit message: Design is ready for order
Parts:
- removed JP16: (no value), pinhead:PINHD-1X8
- removed U$16: PINHD-1X10, adafruit:PINHD-1X10
- removed X2: (no value), con-wago-500:W237-4
- added CR1, CR10, CR11, CR12, CR13, CR14, CR15, CR2, CR3, CR4, CR5, CR6, CR7, CR8, CR9: PESD2CAN24DBZRQ1, TVS_Diode:PESD2CAN24DBZRQ1
- added F10, F11, F12, F13, F14, F15, F2, F3, F4, F5, F6, F7, F8, F9: (no value), Fuse:0154003.DR
- J1: value F-2X18-DIL-100 -> 1888700; device con-headers-jp:F-2X18-DIL-100 -> PheonixContactTerm:1888700
- JP2: device pinhead:PINHD-1X8 -> pinhead:PINHD-2X18
Connections:
- removed net GND: C1.-, C10.-, C11.-, C12.-, C13.-, C14.-, C15.-, C2.-, C3.-, C4.-, C5.-, C6.-, C7.-, C8.-, C9.-, IC1.GND1, IC1.GND2, IC10.GND1, IC10.GND2, IC11.GND1, IC11.GND2, IC12.GND1, IC12.GND2, IC13.GND1, IC13.GND2, IC14.GND1, IC14.GND2, IC15.GND1, IC15.GND2, IC2.GND1, IC2.GND2, IC3.GND1, IC3.GND2, IC4.GND1, IC4.GND2, IC5.GND1, IC5.GND2, IC6.GND1, IC6.GND2, IC7.GND1, IC7.GND2, IC8.GND1, IC8.GND2, IC9.GND1, IC9.GND2, SV1.2, SV1.4, SV10.2, SV10.4, SV11.2, SV11.4, SV12.2, SV12.4, SV13.2, SV13.4, SV14.2, SV14.4, SV15.2, SV15.4, SV2.2, SV2.4, SV3.2, SV3.4, SV4.2, SV4.4, SV5.2, SV5.4, SV6.2, SV6.4, SV7.2, SV7.4, SV8.2, SV8.4, SV9.2, SV9.4, X2-2.KL, X2-3.KL
- removed net N$1: IC11.!SLEEP, JP16.8, R15.2
- removed net N$100: IC9.DIR, J1.24
- removed net N$101: IC10.!SLEEP, J1.26, R10.2
- removed net N$102: IC10.STEP, J1.28
- removed net N$103: IC10.DIR, J1.30
- removed net N$104: IC15.!SLEEP, JP1.4, R11.2
- removed net N$105: IC15.STEP, JP1.3
- removed net N$106: IC15.DIR, JP1.2
- removed net N$13: IC1.DIR, J1.7
- removed net N$14: IC1.STEP, J1.5
- removed net N$15: IC1.!SLEEP, J1.3, R1.2
- removed net N$20: IC2.!SLEEP, J1.9, R2.2
- removed net N$21: IC2.STEP, J1.11
- removed net N$22: IC2.DIR, J1.13
- removed net N$27: IC3.!SLEEP, J1.15, R3.2
- removed net N$28: IC3.STEP, J1.17
- removed net N$29: IC3.DIR, J1.19
- removed net N$4: F1.1, X2-1.KL
- removed net N$42: IC4.!SLEEP, J1.21, R4.2
- removed net N$43: IC4.STEP, J1.23
- removed net N$44: IC4.DIR, J1.25
- removed net N$49: IC5.!SLEEP, J1.27, R5.2
- removed net N$50: IC5.STEP, J1.29
- removed net N$51: IC5.DIR, J1.31
- removed net N$56: IC6.!SLEEP, J1.33, R6.2
- removed net N$57: IC6.STEP, J1.4
- removed net N$58: IC6.DIR, J1.6
- removed net N$7: IC11.STEP, JP16.7
- removed net N$71: IC12.!SLEEP, JP16.5, R14.2
- removed net N$72: IC12.STEP, JP16.4
- removed net N$73: IC12.DIR, JP16.3
- removed net N$78: IC13.!SLEEP, JP16.2, R13.2
- removed net N$79: IC13.STEP, JP16.1
- removed net N$8: IC11.DIR, JP16.6
- removed net N$80: IC13.DIR, JP1.8
- removed net N$85: IC14.!SLEEP, JP1.7, R12.2
- removed net N$86: IC14.STEP, JP1.6
- removed net N$87: IC14.DIR, JP1.5
- removed net N$92: IC7.!SLEEP, J1.8, R7.2
- removed net N$93: IC7.STEP, J1.10
- removed net N$94: IC7.DIR, J1.12
- removed net N$95: IC8.!SLEEP, J1.14, R8.2
- removed net N$96: IC8.STEP, J1.16
- removed net N$97: IC8.DIR, J1.18
- removed net N$98: IC9.!SLEEP, J1.20, R9.2
- removed net N$99: IC9.STEP, J1.22
- removed net VMOT: C1.+, C10.+, C11.+, C12.+, C13.+, C14.+, C15.+, C2.+, C3.+, C4.+, C5.+, C6.+, C7.+, C8.+, C9.+, F1.2, IC1.VMOT, IC10.VMOT, IC11.VMOT, IC12.VMOT, IC13.VMOT, IC14.VMOT, IC15.VMOT, IC2.VMOT, IC3.VMOT, IC4.VMOT, IC5.VMOT, IC6.VMOT, IC7.VMOT, IC8.VMOT, IC9.VMOT
- new net DIR1: IC1.DIR, JP2.7
- new net DIR10: IC10.DIR, JP2.32
- new net DIR11: IC11.DIR, JP3.6
- new net DIR12: IC12.DIR, JP3.3
- new net DIR13: IC13.DIR, JP4.8
- new net DIR14: IC14.DIR, JP4.5
- new net DIR15: IC15.DIR, JP4.2
- new net DIR2: IC2.DIR, JP2.13
- new net DIR3: IC3.DIR, JP2.19
- new net DIR4: IC4.DIR, JP2.25
- new net DIR5: IC5.DIR, JP2.31
- new net DIR6: IC6.DIR, JP2.8
- new net DIR7: IC7.DIR, JP2.14
- new net DIR8: IC8.DIR, JP2.20
- new net DIR9: IC9.DIR, JP2.26
- new net GND1: IC1.GND1, IC10.GND1, IC11.GND1, IC12.GND1, IC13.GND1, IC14.GND1, IC15.GND1, IC2.GND1, IC3.GND1, IC4.GND1, IC5.GND1, IC6.GND1, IC7.GND1, IC8.GND1, IC9.GND1, J1.2, SV1.2, SV1.4, SV10.2, SV10.4, SV11.2, SV11.4, SV12.2, SV12.4, SV13.2, SV13.4, SV14.2, SV14.4, SV15.2, SV15.4, SV2.2, SV2.4, SV3.2, SV3.4, SV4.2, SV4.4, SV5.2, SV5.4, SV6.2, SV6.4, SV7.2, SV7.4, SV8.2, SV8.4, SV9.2, SV9.4
- new net GND2: C1.-, C10.-, C11.-, C12.-, C13.-, C14.-, C15.-, C2.-, C3.-, C4.-, C5.-, C6.-, C7.-, C8.-, C9.-, CR1.3, CR10.3, CR11.3, CR12.3, CR13.3, CR14.3, CR15.3, CR2.3, CR3.3, CR4.3, CR5.3, CR6.3, CR7.3, CR8.3, CR9.3, IC1.GND2, IC10.GND2, IC11.GND2, IC12.GND2, IC13.GND2, IC14.GND2, IC15.GND2, IC2.GND2, IC3.GND2, IC4.GND2, IC5.GND2, IC6.GND2, IC7.GND2, IC8.GND2, IC9.GND2, J1.3
- new net N$182: F1.1, F10.1, F11.1, F12.1, F13.1, F14.1, F15.1, F2.1, F3.1, F4.1, F5.1, F6.1, F7.1, F8.1, F9.1, J1.4
- new net SLP1: IC1.!SLEEP, JP2.3, R1.2
- new net SLP10: IC10.!SLEEP, JP2.28, R10.2
- new net SLP11: IC11.!SLEEP, JP3.8, R11.2
- new net SLP12: IC12.!SLEEP, JP3.5, R12.2
- new net SLP13: IC13.!SLEEP, JP3.2, R13.2
- new net SLP14: IC14.!SLEEP, JP4.7, R14.2
- new net SLP15: IC15.!SLEEP, JP4.4, R15.2
- new net SLP2: IC2.!SLEEP, JP2.9, R2.2
- new net SLP3: IC3.!SLEEP, JP2.15, R3.2
- new net SLP4: IC4.!SLEEP, JP2.21, R4.2
- new net SLP5: IC5.!SLEEP, JP2.27, R5.2
- new net SLP6: IC6.!SLEEP, JP2.4, R6.2
- new net SLP7: IC7.!SLEEP, JP2.10, R7.2
- new net SLP8: IC8.!SLEEP, JP2.16, R8.2
- new net SLP9: IC9.!SLEEP, JP2.22, R9.2
- new net STEP1: IC1.STEP, JP2.5
- new net STEP10: IC10.STEP, JP2.30
- new net STEP11: IC11.STEP, JP3.7
- new net STEP12: IC12.STEP, JP3.4
- new net STEP13: IC13.STEP, JP3.1
- new net STEP14: IC14.STEP, JP4.6
- new net STEP15: IC15.STEP, JP4.3
- new net STEP2: IC2.STEP, JP2.11
- new net STEP3: IC3.STEP, JP2.17
- new net STEP4: IC4.STEP, JP2.23
- new net STEP5: IC5.STEP, JP2.29
- new net STEP6: IC6.STEP, JP2.6
- new net STEP7: IC7.STEP, JP2.12
- new net STEP8: IC8.STEP, JP2.18
- new net STEP9: IC9.STEP, JP2.24
- new net VMOT1: C1.+, CR1.1, CR1.2, F1.2, IC1.VMOT
- new net VMOT10: C10.+, CR10.1, CR10.2, F10.2, IC10.VMOT
- new net VMOT11: C11.+, CR11.1, CR11.2, F11.2, IC11.VMOT
- new net VMOT12: C12.+, CR12.1, CR12.2, F12.2, IC12.VMOT
- new net VMOT13: C13.+, CR13.1, CR13.2, F13.2, IC13.VMOT
- new net VMOT14: C14.+, CR14.1, CR14.2, F14.2, IC14.VMOT
- new net VMOT15: C15.+, CR15.1, CR15.2, F15.2, IC15.VMOT
- new net VMOT2: C2.+, CR2.1, CR2.2, F2.2, IC2.VMOT
- new net VMOT3: C3.+, CR3.1, CR3.2, F3.2, IC3.VMOT
- new net VMOT4: C4.+, CR4.1, CR4.2, F4.2, IC4.VMOT
- new net VMOT5: C5.+, CR5.1, CR5.2, F5.2, IC5.VMOT
- new net VMOT6: C6.+, CR6.1, CR6.2, F6.2, IC6.VMOT
- new net VMOT7: C7.+, CR7.1, CR7.2, F7.2, IC7.VMOT
- new net VMOT8: C8.+, CR8.1, CR8.2, F8.2, IC8.VMOT
- new net VMOT9: C9.+, CR9.1, CR9.2, F9.2, IC9.VMOT
- net 5V: now also J1.1; no longer X2-4.KL
Other:
- moved on the sheet: C1, C10, C11, C12, C13, C14, C15, C2, C3, C4, C5, C6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
